File: PCB/kino-key-midi-part.kicad_sch (KiCad schematic)
At the start: 17 parts, among them J1 AudioJack3, J2 AudioJack3, U6 BAS40DW-04-7-F, U7 TLP2361_TPL_E, U8 CD74HC4050PWR/74HC4050PW

Commit message: [PCB] Update to KiCad 9.0, remove voltage conversion #6
Changed lines of the file:
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@@
 (kicad_sch
-	(version 20231120)
+	(version 20250114)
 	(generator "eeschema")
-	(generator_version "8.0")
+	(generator_version "9.0")
 	(paper "A4")
