File: PCB/kino-key25.kicad_sch (KiCad schematic)
At the start: 107 parts, among them SW1 SW_SPST, SW10 SW_SPST, SW11 SW_SPST, SW12 SW_SPST, SW13 SW_SPST, SW14 SW_SPST, SW15 SW_SPST, SW16 SW_SPST, SW17 SW_SPST, SW18 SW_SPST, SW19 SW_SPST, SW2 SW_SPST, SW20 SW_SPST, SW21 SW_SPST, SW22 SW_SPST, SW23 SW_SPST, SW24 SW_SPST, SW25 SW_SPST, SW26 SW_SPST, SW27 SW_SPST, SW28 SW_SPST, SW29 SW_SPST, SW3 SW_SPST, SW30 SW_SPST, SW31 SW_SPST, SW4 SW_SPST, SW5 SW_SPST, SW6 SW_SPST, SW7 SW_SPST, SW8 SW_SPST, SW9 SW_SPST, U1 74HC165, U2 74HC165, U3 MOUDLE-SEEEDUINO-XIAO, U4 74HC165, U5 74HC165

Commit message: add pdf schematics
Other:
- company: (none) -> kinoshita laboratory
- title: (none) -> kino-key25
Changed lines of the file:
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@@
 	(generator_version "8.0")
 	(paper "A2")
+	(title_block
+		(title "kino-key25")
+		(date "2024-09-17")
+		(rev "20240917")
+		(company "kinoshita laboratory")
+	)
 	(junction
 		(at 355.6 102.87)

Commit message: [PCB] Update to KiCad 9.0, remove voltage conversion #6
Parts:
- added R44: 470, PCM_Resistor_SMD_AKL:R_0603_1608Metric, symbol Device:R
Connections:
- net NEOPIXEL Out: now also R44.1; no longer D1.4 (DI)
- new net: D1.4 (DI), R44.2
Changed lines of the file:
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@@
 (kicad_sch
-	(version 20231120)
+	(version 20250114)
 	(generator "eeschema")
-	(generator_version "8.0")
+	(generator_version "9.0")
 	(paper "A2")
 	(title_block
@@
 		(company "kinoshita laboratory")
 	)
+	(text "D4: reserved"
+		(exclude_from_sim no)
+		(at 124.46 177.8 0)
+		(effects
+			(font
+				(size 1.27 1.27)
+			)
+		)
+	)
 	(junction
 		(at 355.6 102.87)
@@
 	(wire
 		(pts
+			(xy 304.8 38.1) (xy 322.58 38.1)
+		)
+		(stroke
+			(width 0)
+			(type default)
+		)
+	)
+	(wire
+		(pts
 			(xy 185.42 364.49) (xy 187.96 364.49)
 		)
@@
 	(wire
 		(pts
+			(xy 330.2 38.1) (xy 340.36 38.1)
+		)
+		(stroke
+			(width 0)
+			(type default)
+		)
+	)
+	(wire
+		(pts
 			(xy 435.61 358.14) (xy 435.61 364.49)
 		)
@@
 		)
 	)
-	(text "D4: reserved"
-		(exclude_from_sim no)
-		(at 124.46 177.8 0)
-		(effects
-			(font
-				(size 1.27 1.27)
-			)
-		)
-	)
 	(global_label "CP"
 		(shape input)
@@
 	(global_label "NEOPIXEL Out"
 		(shape input)
-		(at 340.36 38.1 180)
+		(at 304.8 38.1 180)
 		(fields_autoplaced yes)
 		(effects
@@
 		)
 		(property "Intersheetrefs" "${INTERSHEET_REFS}"
-			(at 324.1306 38.1 0)
+			(at 288.5706 38.1 0)
 			(effects
 				(font
@@
 	(symbol
 		(lib_id "Device:R")
+		(at 326.39 38.1 90)
+		(unit 1)
+		(exclude_from_sim no)
+		(in_bom yes)
+		(on_board yes)
+		(dnp no)
+		(fields_autoplaced yes)
+		(property "Reference" "R44"
+			(at 326.39 31.75 90)
+			(effects
+				(font
+					(size 1.27 1.27)
+				)
+			)
+		)
+		(property "Value" "470"
+			(at 326.39 34.29 90)
+			(effects
+				(font
+					(size 1.27 1.27)
+				)
+			)
+		)
+		(property "Footprint" "PCM_Resistor_SMD_AKL:R_0603_1608Metric"
+			(at 326.39 39.878 90)
+			(effects
+				(font
+					(size 1.27 1.27)
+				)
+				(hide yes)
+			)
+		)
+		(property "Datasheet" "~"
+			(at 326.39 38.1 0)
+			(effects
+				(font
+					(size 1.27 1.27)
+				)
+				(hide yes)
+			)
+		)
+		(property "Description" "Resistor"
+			(at 326.39 38.1 0)
+			(effects
+				(font
+					(size 1.27 1.27)
+				)
+				(hide yes)
+			)
+		)
+		(property "LCSC" "C23179"
+			(at 326.39 38.1 90)
+			(effects
+				(font
+					(size 1.27 1.27)
+				)
+				(hide yes)
+			)
+		)
+		(pin "1"
+		)
+		(pin "2"
+		)
+		(instances
+			(project ""
+				(path "/643d6f24-7dc5-473d-9f3e-1d00b489c9c7"
+					(reference "R44")
+					(unit 1)
+				)
+			)
+		)
+	)
+	(symbol
+		(lib_id "Device:R")
 		(at 138.43 177.8 0)
 		(mirror x)
@@
 		(at 488.95 199.39)
 		(size 25.4 16.51)
+		(exclude_from_sim no)
+		(in_bom yes)
+		(on_board yes)
+		(dnp no)
 		(fields_autoplaced yes)
 		(stroke
@@
 		)
 	)
+	(embedded_fonts no)
 )
